Commit message: Update modelo.urdf

File: Practicas/P1/modelo.urdf (robot description, URDF)
Before this commit: robot Practica-1, 7 links, 6 joints
Joints:
- joint forearm_joint: limit (none) -> lower=-2.587 upper=2.587 effort=10.0 velocity=0.5
- joint pinza_joint: limit (none) -> lower=0 upper=0 effort=10.0 velocity=0.5
- joint shoulder_joint: limit (none) -> lower=-3.14 upper=3.14 effort=10.0 velocity=0.5
- joint trunk_joint: limit (none) -> lower=0 upper=0 effort=10.0 velocity=0.5
- joint world_joint: limit (none) -> lower=0 upper=0 effort=10.0 velocity=0.5
